File: Breaking_disc_control_unit/Breaking_disc_control_unit.kicad_pcb (KiCad board)
At the start: 2 copper layers, 69 parts, among them J1 Conn_02x05_Odd_Even, J2 Conn_02x03_Odd_Even, J3 Conn_01x02, J4 Conn_01x04, J5 Conn_01x03, SW1 SW_Push, U1 MKW31Z256VHT4, U2 TLV4964, U3 MMA8452Q, U4 MPL3115A2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

Commit message: Layout fast fertig!
Parts:
- removed the REF** at (161.6, 85.2)
- moved C35 6.41 mm to (165.8, 90.9)
- moved C20 4.74 mm to (106.2, 95.9), turned to 270 degrees
- moved C27 4.23 mm to (166.8, 92.8)
- moved D1 4.11 mm to (110.3, 92.5), turned to 0 degrees
- moved C19 3.09 mm to (109.8, 87.4), turned to 180 degrees
- moved R5 2.62 mm to (108.4, 102.6)
- moved C16 2.48 mm to (104.5, 98.8), turned to 270 degrees
- moved R8 2.07 mm to (96.9, 100.3), turned to 0 degrees
- moved R2 1.29 mm to (140.4, 99.5)
- moved C2 1.25 mm to (148.3, 84.1)
- moved C22 1.25 mm to (117.4, 96.5)
- moved C30 1.15 mm to (162.2, 81.6), turned to 180 degrees
- moved C34 1.13 mm to (162.2, 84.0), turned to 180 degrees
- moved C17 1.11 mm to (106.2, 100.0)
- moved U5 0.90 mm to (111.5, 98.1)
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Routing:
- net GND: track 0.00 -> 141.0 mm, vias 0 -> 16
- net +BATT: track 1.63 -> 91.9 mm, vias 0 -> 4
- net Net-(R6-Pad2): track 0.00 -> 79.5 mm, vias 0 -> 2
- net +3V3: track 33.8 -> 101.9 mm, vias 1 -> 10
- net I2C_INT_21: track 4.13 -> 27.4 mm, vias 0 -> 2
- net VSOURCE: track 18.2 -> 41.4 mm, vias 0 -> 2
- net I2C_INT_22: track 3.13 -> 26.3 mm, vias 0 -> 2
- net Net-(C17-Pad1): track 0.00 -> 19.0 mm
- net Net-(D1-Pad2): track 0.00 -> 13.5 mm
- net Net-(C16-Pad1): track 0.00 -> 12.8 mm
- net I2C_SCL: track 11.8 -> 21.8 mm, vias 2 -> 3
- net I2C_SDA: track 13.9 -> 22.8 mm, vias 2 -> 3
- net XTAL_32MHZ: track 9.15 -> 12.8 mm
- net Net-(R5-Pad2): track 0.00 -> 3.42 mm
- net Net-(L1-Pad2): track 0.00 -> 3.35 mm
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- added copper zone on F.Cu, net +3V3
- added copper zone on B.Cu, net GND
- added copper zone on F.Cu, net GND
