File: Breaking_disc_control_unit/Breaking_disc_control_unit.kicad_pcb (KiCad board)
At the start: 2 copper layers, 68 parts, among them J1 Conn_02x05_Odd_Even, J2 Conn_02x03_Odd_Even, J3 Conn_01x02, J4 Conn_01x04, J5 Conn_01x03, SW1 SW_Push, U1 MKW31Z256VHT4, U2 TLV4964, U3 MMA8452Q, U4 MPL3115A2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

Commit message: LAYOUT FERTIG!!! NOT REVIEWED YET!
Parts:
- moved C26 0.75 mm to (166.3, 95.0)
- moved C12 0.65 mm to (137.2, 85.6)
- moved C34 0.50 mm to (162.2, 84.5)
- moved C35 0.43 mm to (165.7, 90.5)
- moved J1 0.42 mm to (139.3, 86.7)
- moved L2 0.40 mm to (161.6, 83.3)
- moved C30 0.30 mm to (162.2, 81.9)
- moved C15 0.25 mm to (145.2, 100.6)
- moved AE1 0.25 mm to (161.6, 81.0)
- moved Y1 0.25 mm to (162.3, 93.8)
Routing:
- net GND: track 141.0 -> 233.4 mm, vias 16 -> 45
- net +3V3: track 101.9 -> 180.8 mm
- net I2C_SDA: track 22.8 -> 25.3 mm
- net UART0_TX: track 18.3 -> 16.8 mm
- net EXTAL_32MHZ: track 11.8 -> 13.2 mm
- net SPI1_SCK_EXT: track 40.8 -> 39.4 mm
- net UART0_RX: track 26.6 -> 25.2 mm
- net SPI1_PCS0_EXT: track 36.4 -> 35.5 mm
- net SWD_CLK: track 5.63 -> 4.97 mm
- net I2C_INT_22: track 26.3 -> 25.7 mm
- net Net-(C34-Pad2): track 11.1 -> 10.4 mm
- net SM_BIN2/BENBL: track 46.4 -> 45.8 mm
- net SM_BIN1/BP: track 43.2 -> 42.6 mm
- net SM_AIN2/AENBL: track 43.2 -> 42.6 mm
- net (no net): vias 6 -> 1

Commit message: LAYOUT REVIEWD AND SENT!
Routing:
- net GND: track 233.4 -> 270.6 mm, vias 45 -> 58
- net +3V3: track 180.8 -> 170.1 mm
- net I2C_INT_22: track 25.7 -> 26.6 mm
- net (no net): track 0.00 -> 0.02 mm, vias 1 -> 0
Other:
- net class Power: clearance 0.3 -> 0.2; trace_width 0.4 -> 0.3
