File: Breaking_disc_control_unit/Breaking_disc_control_unit.kicad_pcb (KiCad board)
At the start: 2 copper layers, 68 parts, among them J1 Conn_02x05_Odd_Even, J2 Conn_02x03_Odd_Even, J3 Conn_01x02, J4 Conn_01x04, J5 Conn_01x03, SW1 SW_Push, U1 MKW31Z256VHT4, U2 TLV4964, U3 MMA8452Q, U4 MPL3115A2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

Commit message: Gerberfiles HSLU
Other:
- board outline added: 88 x 34 mm
Changed lines of the file:
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@@
     (links 206)
     (no_connects 0)
-    (area 0 0 0 0)
+    (area 66.750001 56.050686 176.571429 115.099527)
     (thickness 0.8)
-    (drawings 11)
+    (drawings 12)
     (tracks 892)
     (zones 0)
@@
     (trace_min 0.2)
     (segment_width 0.2)
-    (edge_width 0.1)
+    (edge_width 0.2)
     (via_size 0.75)
     (via_drill 0.4)
@@
     )
   )
+  (dimension 37.550008 (width 0.3) (layer F.Fab)
+    (gr_text "37.550 mm" (at 101.341595 61.03902 0.03814631894) (layer F.Fab)
+      (effects (font (size 1.5 1.5) (thickness 0.3)))
+    )
+    (feature1 (pts (xy 82.575 73.675) (xy 82.565696 59.701521)))
+    (feature2 (pts (xy 120.125 73.65) (xy 120.115696 59.676521)))
+    (crossbar (pts (xy 120.117494 62.37652) (xy 82.567494 62.40152)))
+    (arrow1a (pts (xy 82.567494 62.40152) (xy 83.693607 61.814349)))
+    (arrow1b (pts (xy 82.567494 62.40152) (xy 83.694388 62.987191)))
+    (arrow2a (pts (xy 120.117494 62.37652) (xy 118.9906 61.790849)))
+    (arrow2b (pts (xy 120.117494 62.37652) (xy 118.991381 62.963691)))
+  )
   (dimension 80.000016 (width 0.3) (layer F.Fab)
     (gr_text "80.000 mm" (at 126.207655 113.724526 0.03580985753) (layer F.Fab)
@@
     (arrow2b (pts (xy 79 101.5) (xy 78.413579 100.373496)))
   )
-  (gr_line (start 83 104.925) (end 170.6 104.925) (angle 90) (layer F.Fab) (width 0.2))
+  (gr_line (start 83 104.925) (end 170.6 104.925) (angle 90) (layer Edge.Cuts) (width 0.2))
   (gr_text "Breaking disc control unit V1.0\nRobert Näger" (at 91.55 76.3 90) (layer B.SilkS)
     (effects (font (size 1 1) (thickness 0.25)) (justify left mirror))
   )
-  (gr_line (start 170.6 104.925) (end 170.6 70.875) (angle 90) (layer F.Fab) (width 0.2))
-  (gr_line (start 82.575 104.925) (end 82.575 70.875) (angle 90) (layer F.Fab) (width 0.2))
-  (gr_line (start 82.825 70.875) (end 170.6 70.875) (angle 90) (layer F.Fab) (width 0.2))
+  (gr_line (start 170.6 104.925) (end 170.6 70.875) (angle 90) (layer Edge.Cuts) (width 0.2))
+  (gr_line (start 82.575 104.925) (end 82.575 70.875) (angle 90) (layer Edge.Cuts) (width 0.2))
+  (gr_line (start 82.825 70.875) (end 170.6 70.875) (angle 90) (layer Edge.Cuts) (width 0.2))
   (segment (start 161.75697 89.2) (end 161.647987 89.091017) (width 0.5) (layer F.Cu) (net 1))
   (segment (start 163.7 89.2) (end 161.75697 89.2) (width 0.5) (layer F.Cu) (net 1))
